File: PCB/PixelWave.kicad_sch (KiCad schematic)
At the start: 663 parts, among them J1 Conn_01x06, Q1 STL6P3LLH6, Q2 STL6P3LLH6, U1 HT7533-1, U3 ESP32-S3-WROOM-1, U4 XL4016, U5 STUSB4500QTR

Commit message: Optimize traces and switch inductor
Parts:
- C317, C321: footprint Capacitor_THT:C_Radial_D10.0mm_H16.0mm_P5.00mm -> Capacitor_THT:CP_Radial_D10.0mm_P5.00mm; symbol Device:C -> Device:C_Polarized
- L1: footprint Inductor_SMD:L_Pulse_PA4349 -> Components:IND-TH_L33.0-W15.6-P15.00-D1.5
Changed lines of the file:
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@@
 	)
 	(symbol
-		(lib_id "Device:C")
+		(lib_id "Device:C_Polarized")
 		(at 391.16 38.1 0)
 		(unit 1)
@@
 			)
 		)
-		(property "Footprint" "Capacitor_THT:C_Radial_D10.0mm_H16.0mm_P5.00mm"
+		(property "Footprint" "Capacitor_THT:CP_Radial_D10.0mm_P5.00mm"
 			(at 392.1252 41.91 0)
 			(effects
@@
 			)
 		)
-		(property "Description" "Unpolarized capacitor"
+		(property "Description" "Polarized capacitor"
 			(at 391.16 38.1 0)
 			(effects
@@
 	)
 	(symbol
-		(lib_id "Device:C")
+		(lib_id "Device:C_Polarized")
 		(at 294.64 38.1 0)
 		(unit 1)
@@
 			)
 		)
-		(property "Footprint" "Capacitor_THT:C_Radial_D10.0mm_H16.0mm_P5.00mm"
+		(property "Footprint" "Capacitor_THT:CP_Radial_D10.0mm_P5.00mm"
 			(at 295.6052 41.91 0)
 			(effects
@@
 			)
 		)
-		(property "Description" "Unpolarized capacitor"
+		(property "Description" "Polarized capacitor"
 			(at 294.64 38.1 0)
 			(effects
@@
 			)
 		)
-		(property "Footprint" "Inductor_SMD:L_Pulse_PA4349"
+		(property "Footprint" "Components:IND-TH_L33.0-W15.6-P15.00-D1.5"
 			(at 365.76 34.29 0)
 			(effects

Commit message: wjdhasjkd
Parts:
- D5: footprint Package_TO_SOT_THT:TO-220-2_Horizontal_TabDown -> Package_TO_SOT_THT:TO-220-3_Horizontal_TabDown
Changed lines of the file:
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@@
 			)
 		)
-		(property "Footprint" "Package_TO_SOT_THT:TO-220-2_Horizontal_TabDown"
+		(property "Footprint" "Package_TO_SOT_THT:TO-220-3_Horizontal_TabDown"
 			(at 353.06 38.1 0)
 			(effects

Commit message: asdjoa
Parts:
- U4: footprint Package_TO_SOT_SMD:TO-263-5_TabPin3 -> Components:TO-220-5L_L10.2-W4.5-P1.71-L
Changed lines of the file:
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@@
 			)
 		)
-		(property "Footprint" "Package_TO_SOT_SMD:TO-263-5_TabPin3"
+		(property "Footprint" "Components:TO-220-5L_L10.2-W4.5-P1.71-L"
 			(at 356.87 44.45 0)
 			(effects

Commit message: fix: footprints
Parts:
- removed D1, D4: ESDA25P35, Components:TVS_ESDA25P35-1U1M, symbol ESDA25P35:ESDA25P35-1U1M
- added D1, D4: ~, Components:DFN1610-2_L1.6-W1.0-P1.05-RD, symbol C1974707:ESDA25P35-1U1M
- D2: footprint Diode_SMD:D_SOD-123 -> Diode_SMD:D_SOD-323
Connections:
- net C_Vsnk: now also D4.1
- net GND: now also D1.2, D4.2
- net VBUS: now also D1.1

Commit message: fix: more footprint issues
Parts:
- R14: footprint Resistor_SMD:R_1206_3216Metric -> Resistor_SMD:R_0805_2012Metric
Changed lines of the file:
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@@
 			)
 		)
-		(property "Footprint" "Resistor_SMD:R_1206_3216Metric"
+		(property "Footprint" "Resistor_SMD:R_0805_2012Metric"
 			(at 197.358 55.88 90)
 			(effects

Commit message: start v2
Parts:
- removed C311: 4.7uF, Capacitor_SMD:C_1206_3216Metric, symbol Device:C
- removed C315: 1uF, Capacitor_SMD:C_1206_3216Metric, symbol Device:C
- removed C316: 100nF, Capacitor_SMD:C_1206_3216Metric, symbol Device:C
- removed C317: 470uF/50V, Capacitor_THT:CP_Radial_D10.0mm_P5.00mm, symbol Device:C_Polarized
- removed C318, C319, C320: 1uF, Capacitor_SMD:C_0805_2012Metric, symbol Device:C
- removed C321: 1000uF, Capacitor_THT:CP_Radial_D10.0mm_P5.00mm, symbol Device:C_Polarized
- removed D1, D4: ~, Components:DFN1610-2_L1.6-W1.0-P1.05-RD, symbol C1974707:ESDA25P35-1U1M
- removed D2: 1N5819W, Diode_SMD:D_SOD-323, symbol Device:D_Schottky
- removed D3: ESDA5V3L, Package_TO_SOT_SMD:SOT-23-3, symbol Power_Protection:ESDA5V3L
- removed D5: MBR1545, Package_TO_SOT_THT:TO-220-3_Horizontal_TabDown, symbol Device:D_Schottky
- removed L1: 47uH/12A, Components:IND-TH_L33.0-W15.6-P15.00-D1.5, symbol XR106125TS470MV1L5:XR106125TS470MV1L5
- removed Q1, Q2: STL6P3LLH6, Components:STL6P3LLH6, symbol STL6P3LLH6:STL6P3LLH6
- removed R1: 470, Resistor_SMD:R_1206_3216Metric, symbol Device:R
- removed R10, R15, R6: 100k, Resistor_SMD:R_1206_3216Metric, symbol Device:R
- removed R11, R12: NC, Resistor_SMD:R_1206_3216Metric, symbol Device:R
- removed R13, R7: 10k, Resistor_SMD:R_1206_3216Metric, symbol Device:R
- removed R14: 22k, Resistor_SMD:R_0805_2012Metric, symbol Device:R
- removed R16: 100, Resistor_SMD:R_1206_3216Metric, symbol Device:R
- removed R17, R4: 1k, Resistor_SMD:R_1206_3216Metric, symbol Device:R
- removed R18, R5, R9: 4.7k, Resistor_SMD:R_1206_3216Metric, symbol Device:R
- removed R8: 3.3k, Resistor_SMD:R_1206_3216Metric, symbol Device:R
- removed U2: ~, Components:USB-C-SMD_G-SWITCH_GT-USB-7010ASV, symbol USB_C:GT-USB-7010ASV
- removed U4: XL4016, Components:TO-220-5L_L10.2-W4.5-P1.71-L, symbol Regulator_Switching:XL4015
- removed U5: STUSB4500QTR, Package_DFN_QFN:QFN-24-1EP_4x4mm_P0.5mm_EP2.7x2.7mm, symbol Interface_USB:STUSB4500QTR
- added C311: 470uF, symbol Device:C_Polarized
- added D1: LED, symbol Device:LED
- added J1: XT60, Connector_AMASS:AMASS_XT60-F_1x02_P7.20mm_Vertical, symbol Connector_Generic:Conn_01x02
- added J3: Conn_01x02, symbol Connector_Generic:Conn_01x02
- added J4: Conn_01x04, symbol Connector_Generic:Conn_01x04
- added U2: XL4016, Package_TO_SOT_SMD:TO-263-5_TabPin3, symbol Regulator_Switching:XL4015
- C312, C313: footprint Capacitor_SMD:C_1206_3216Metric -> (none)
- C314: value 1uF -> 105; footprint Capacitor_SMD:C_1206_3216Metric -> (none)
- J2: renamed from J1; symbol Connector_Generic:Conn_01x06 -> Connector_Generic:Conn_01x07
Connections:
- net C_Vsnk is gone; now on net VCC: U1.2 (VIN)
- net +3V3: now also D1.2 (A)
- net +5V: now also J2.7 (Pin_7), J4.1 (Pin_1); no longer C1.1, C10.1, C100.1, C101.1, C102.1, C103.1, C104.1, C105.1, C106.1, C107.1, C108.1, C109.1, C11.1, C110.1, C111.1, C112.1, C113.1, C114.1, C115.1, C116.1, C117.1, C118.1, C119.1, C12.1, C120.1, C121.1, C122.1, C123.1, C124.1, C125.1, C126.1, C127.1, C128.1, C129.1, C13.1, C130.1, C131.1, C132.1, C133.1, C134.1, C135.1, C136.1, C137.1, C138.1, C139.1, C14.1, C140.1, C141.1, C142.1, C143.1, C144.1, C145.1, C146.1, C147.1, C148.1, C149.1, C15.1, C150.1, C151.1, C152.1, C153.1, C154.1, C155.1, C156.1, C157.1, C158.1, C159.1, C16.1, C160.1, C161.1, C162.1, C163.1, C164.1, C165.1, C166.1, C167.1, C168.1, C169.1, C17.1, C170.1, C171.1, C172.1, C173.1, C174.1, C175.1, C176.1, C177.1, C178.1, C179.1, C18.1, C180.1, C181.1, C182.1, C183.1, C184.1, C185.1, C186.1, C187.1, C188.1, C189.1, C19.1, C190.1, C191.1, C192.1, C193.1, C194.1, C195.1, C196.1, C197.1, C198.1, C199.1, C2.1, C20.1, C200.1, C201.1, C202.1, C203.1, C204.1, C205.1, C206.1, C207.1, C208.1, C209.1, C21.1, C210.1, C211.1, C212.1, C213.1, C214.1, C215.1, C216.1, C217.1, C218.1, C219.1, C22.1, C220.1, C221.1, C222.1, C223.1, C224.1, C225.1, C226.1, C227.1, C228.1, C229.1, C23.1, C230.1, C231.1, C232.1, C233.1, C234.1, C235.1, C236.1, C237.1, C238.1, C239.1, C24.1, C240.1, C241.1, C242.1, C243.1, C244.1, C245.1, C246.1, C247.1, C248.1, C249.1, C25.1, C250.1, C251.1, C252.1, C253.1, C254.1, C255.1, C256.1, C257.1, C258.1, C259.1, C26.1, C260.1, C261.1, C262.1, C263.1, C264.1, C265.1, C266.1, C267.1, C268.1, C269.1, C27.1, C270.1, C271.1, C272.1, C273.1, C274.1, C275.1, C276.1, C277.1, C278.1, C279.1, C28.1, C280.1, C281.1, C282.1, C283.1, C284.1, C285.1, C286.1, C287.1, C288.1, C289.1, C29.1, C290.1, C291.1, C292.1, C293.1, C294.1, C295.1, C296.1, C297.1, C298.1, C299.1, C3.1, C30.1, C300.1, C301.1, C302.1, C303.1, C304.1, C305.1, C306.1, C307.1, C308.1, C309.1, C31.1, C310.1, C32.1, C33.1, C34.1, C35.1, C36.1, C37.1, C38.1, C39.1, C4.1, C40.1, C41.1, C42.1, C43.1, C44.1, C45.1, C46.1, C47.1, C48.1, C49.1, C5.1, C50.1, C51.1, C52.1, C53.1, C54.1, C55.1, C56.1, C57.1, C58.1, C59.1, C6.1, C60.1, C61.1, C62.1, C63.1, C64.1, C65.1, C66.1, C67.1, C68.1, C69.1, C7.1, C70.1, C71.1, C72.1, C73.1, C74.1, C75.1, C76.1, C77.1, C78.1, C79.1, C8.1, C80.1, C81.1, C82.1, C83.1, C84.1, C85.1, C86.1, C87.1, C88.1, C89.1, C9.1, C90.1, C91.1, C92.1, C93.1, C94.1, C95.1, C96.1, C97.1, C98.1, C99.1, D100.4 (VDD), D101.4 (VDD), D102.4 (VDD), D103.4 (VDD), D104.4 (VDD), D105.4 (VDD), D106.4 (VDD), D107.4 (VDD), D108.4 (VDD), D109.4 (VDD), D110.4 (VDD), D111.4 (VDD), D112.4 (VDD), D113.4 (VDD), D114.4 (VDD), D115.4 (VDD), D116.4 (VDD), D117.4 (VDD), D118.4 (VDD), D119.4 (VDD), D120.4 (VDD), D121.4 (VDD), D122.4 (VDD), D123.4 (VDD), D124.4 (VDD), D125.4 (VDD), D126.4 (VDD), D127.4 (VDD), D128.4 (VDD), D129.4 (VDD), D13.4 (VDD), D130.4 (VDD), D131.4 (VDD), D132.4 (VDD), D133.4 (VDD), D134.4 (VDD), D135.4 (VDD), D136.4 (VDD), D137.4 (VDD), D138.4 (VDD), D139.4 (VDD), D14.4 (VDD), D140.4 (VDD), D141.4 (VDD), D142.4 (VDD), D143.4 (VDD), D144.4 (VDD), D145.4 (VDD), D146.4 (VDD), D147.4 (VDD), D148.4 (VDD), D149.4 (VDD), D15.4 (VDD), D150.4 (VDD), D151.4 (VDD), D152.4 (VDD), D153.4 (VDD), D154.4 (VDD), D155.4 (VDD), D156.4 (VDD), D157.4 (VDD), D158.4 (VDD), D159.4 (VDD), D16.4 (VDD), D160.4 (VDD), D161.4 (VDD), D162.4 (VDD), D163.4 (VDD), D164.4 (VDD), D165.4 (VDD), D166.4 (VDD), D167.4 (VDD), D168.4 (VDD), D169.4 (VDD), D17.4 (VDD), D170.4 (VDD), D171.4 (VDD), D172.4 (VDD), D173.4 (VDD), D174.4 (VDD), D175.4 (VDD), D176.4 (VDD), D177.4 (VDD), D178.4 (VDD), D179.4 (VDD), D18.4 (VDD), D180.4 (VDD), D181.4 (VDD), D182.4 (VDD), D183.4 (VDD)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
- net GND: now also C312.2, C311.2, D1.1 (K), J1.1 (Pin_1), J4.4 (Pin_4); no longer C312.1, C314.2
- net USB_DM: now also J4.3 (Pin_3)
- net USB_DP: now also J4.2 (Pin_2)
- net VCC: now reaches C313.1
- net VCC: now also C1.1, C10.1, C100.1, C101.1, C102.1, C103.1, C104.1, C105.1, C106.1, C107.1, C108.1, C109.1, C11.1, C110.1, C111.1, C112.1, C113.1, C114.1, C115.1, C116.1, C117.1, C118.1, C119.1, C12.1, C120.1, C121.1, C122.1, C123.1, C124.1, C125.1, C126.1, C127.1, C128.1, C129.1, C13.1, C130.1, C131.1, C132.1, C133.1, C134.1, C135.1, C136.1, C137.1, C138.1, C139.1, C14.1, C140.1, C141.1, C142.1, C143.1, C144.1, C145.1, C146.1, C147.1, C148.1, C149.1, C15.1, C150.1, C151.1, C152.1, C153.1, C154.1, C155.1, C156.1, C157.1, C158.1, C159.1, C16.1, C160.1, C161.1, C162.1, C163.1, C164.1, C165.1, C166.1, C167.1, C168.1, C169.1, C17.1, C170.1, C171.1, C172.1, C173.1, C174.1, C175.1, C176.1, C177.1, C178.1, C179.1, C18.1, C180.1, C181.1, C182.1, C183.1, C184.1, C185.1, C186.1, C187.1, C188.1, C189.1, C19.1, C190.1, C191.1, C192.1, C193.1, C194.1, C195.1, C196.1, C197.1, C198.1, C199.1, C2.1, C20.1, C200.1, C201.1, C202.1, C203.1, C204.1, C205.1, C206.1, C207.1, C208.1, C209.1, C21.1, C210.1, C211.1, C212.1, C213.1, C214.1, C215.1, C216.1, C217.1, C218.1, C219.1, C22.1, C220.1, C221.1, C222.1, C223.1, C224.1, C225.1, C226.1, C227.1, C228.1, C229.1, C23.1, C230.1, C231.1, C232.1, C233.1, C234.1, C235.1, C236.1, C237.1, C238.1, C239.1, C24.1, C240.1, C241.1, C242.1, C243.1, C244.1, C245.1, C246.1, C247.1, C248.1, C249.1, C25.1, C250.1, C251.1, C252.1, C253.1, C254.1, C255.1, C256.1, C257.1, C258.1, C259.1, C26.1, C260.1, C261.1, C262.1, C263.1, C264.1, C265.1, C266.1, C267.1, C268.1, C269.1, C27.1, C270.1, C271.1, C272.1, C273.1, C274.1, C275.1, C276.1, C277.1, C278.1, C279.1, C28.1, C280.1, C281.1, C282.1, C283.1, C284.1, C285.1, C286.1, C287.1, C288.1, C289.1, C29.1, C290.1, C291.1, C292.1, C293.1, C294.1, C295.1, C296.1, C297.1, C298.1, C299.1, C3.1, C30.1, C300.1, C301.1, C302.1, C303.1, C304.1, C305.1, C306.1, C307.1, C308.1, C309.1, C31.1, C310.1, C312.1, C314.1, C32.1, C33.1, C34.1, C35.1, C36.1, C37.1, C38.1, C39.1, C4.1, C40.1, C41.1, C42.1, C43.1, C44.1, C45.1, C46.1, C47.1, C48.1, C49.1, C5.1, C50.1, C51.1, C52.1, C53.1, C54.1, C55.1, C56.1, C57.1, C58.1, C59.1, C6.1, C60.1, C61.1, C62.1, C63.1, C64.1, C65.1, C66.1, C67.1, C68.1, C69.1, C7.1, C70.1, C71.1, C72.1, C73.1, C74.1, C75.1, C76.1, C77.1, C78.1, C79.1, C8.1, C80.1, C81.1, C82.1, C83.1, C84.1, C85.1, C86.1, C87.1, C88.1, C89.1, C9.1, C90.1, C91.1, C92.1, C93.1, C94.1, C95.1, C96.1, C97.1, C98.1, C99.1, D100.4 (VDD), D101.4 (VDD), D102.4 (VDD), D103.4 (VDD), D104.4 (VDD), D105.4 (VDD), D106.4 (VDD), D107.4 (VDD), D108.4 (VDD), D109.4 (VDD), D110.4 (VDD), D111.4 (VDD), D112.4 (VDD), D113.4 (VDD), D114.4 (VDD), D115.4 (VDD), D116.4 (VDD), D117.4 (VDD), D118.4 (VDD), D119.4 (VDD), D120.4 (VDD), D121.4 (VDD), D122.4 (VDD), D123.4 (VDD), D124.4 (VDD), D125.4 (VDD), D126.4 (VDD), D127.4 (VDD), D128.4 (VDD), D129.4 (VDD), D13.4 (VDD), D130.4 (VDD), D131.4 (VDD), D132.4 (VDD), D133.4 (VDD), D134.4 (VDD), D135.4 (VDD), D136.4 (VDD), D137.4 (VDD), D138.4 (VDD), D139.4 (VDD), D14.4 (VDD), D140.4 (VDD), D141.4 (VDD), D142.4 (VDD), D143.4 (VDD), D144.4 (VDD), D145.4 (VDD), D146.4 (VDD), D147.4 (VDD), D148.4 (VDD), D149.4 (VDD), D15.4 (VDD), D150.4 (VDD), D151.4 (VDD), D152.4 (VDD), D153.4 (VDD), D154.4 (VDD), D155.4 (VDD), D156.4 (VDD), D157.4 (VDD), D158.4 (VDD), D159.4 (VDD), D16.4 (VDD), D160.4 (VDD), D161.4 (VDD), D162.4 (VDD), D163.4 (VDD), D164.4 (VDD), D165.4 (VDD), D166.4 (VDD), D167.4 (VDD), D168.4 (VDD), D169.4 (VDD), D17.4 (VDD), D170.4 (VDD), D171.4 (VDD), D172.4 (VDD), D173.4 (VDD), D174.4 (VDD), D175.4 (VDD), D176.4 (VDD), D177.4 (VDD), D178.4 (VDD), D179.4 (VDD), D18.4 (VDD), D180.4 (VDD), D181.4 (VDD)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
- new net: C314.2, U2.4 (VC)
- no-connect marks 30 -> 23
Other:
- moved on the sheet: SW1, U1, U3
